File: kicad/board-layout/cablight.kicad_pcb (KiCad board)
At the start: 2 copper layers, 140 x 42 mm, 19 parts, among them J1 Screw_Term_1x2_2.54mm, J1 Screw_Terminal_01x02, J2 Screw_Term_1x2_2.54mm, J2 Screw_Terminal_01x02, J3 Screw_Terminal_HCSR04, Q1 IRLB8721PBF, SW1 Rotary Encoder (Quadrature) P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, SW2 SW_SPST

Commit message: update board layout
Parts:
- removed the J1 at (162.2, 106.2)
- removed the J1 at (2.59, 6.40)
- removed the J2 at (11.2, 6.40)
- removed the J2 at (162.2, 116.3)
- removed the REF** at (125.0, 84.5)
- removed SW2: SW_SPST, user:CUI_SPDT_500mA_3mm
- added ?: Hole10mm, user:Hole10mm, F.Cu at (136.0, 104.0)
- added D1: 1N5817, Diode_THT:D_DO-41_SOD81_P2.54mm_Vertical_KathodeUp, F.Cu at (191.6, 83.3)
- added J1: Screw_Term_1x2_2.54mm, user:2xTermBlock_254mm, F.Cu at (156.1, 106.2)
- added J2: Screw_Term_1x2_2.54mm, user:2xTermBlock_254mm, F.Cu at (156.1, 116.3)
- added M3: MountingHole_3.2mm_M3_ISO14580_Pad_TopOnly, user:MountingHole_3.2mm_M3_ISO14580_Pad_TopOnly, B.Cu at (182.9, 111.2)
- added REF**: MountingHole_2.7mm_M2.5_ISO7380_Pad_Heated_Insert, user:MountingHole_2.7mm_M2.5_ISO7380_Pad_Heated_Insert, F.Cu at (123.0, 86.0)
- added SW3: switch_SPDT_SLW_121586, user:CUI_SPDT_500mA_3mm, F.Cu at (174.6, 85.8)
- added TP1: GND, TestPoint:TestPoint_Plated_Hole_D2.0mm, F.Cu at (116.4, 92.0)
- added TP2: 5V, TestPoint:TestPoint_Plated_Hole_D2.0mm, F.Cu at (132.5, 91.8)
- REF** (x3): value MountingHole_2.7mm_M2.5_ISO7380_Pad -> MountingHole_2.7mm_M2.5_ISO7380_Pad_Heated_Insert; footprint user:MountingHole_2.7mm_M2.5_ISO7380_Pad -> user:MountingHole_2.7mm_M2.5_ISO7380_Pad_Heated_Insert
- SW1: footprint user:Bourns-PEC11R-4220F-S0024-0-0-0 -> user:Bourns-PEC11R
- moved REF** 10.0 mm to (115.0, 117.0)
- moved R4 8.92 mm to (179.5, 96.0)
- moved R5 8.92 mm to (175.7, 96.0)
- moved Pololu_5V_1 8.70 mm to (154.8, 88.4)
- moved REF** 8.25 mm to (235.0, 109.0)
- moved Q1 8.06 mm to (165.6, 108.7)
- moved R1 6.16 mm to (225.9, 117.6)
- moved R2 6.16 mm to (225.9, 112.5)
- moved R3 6.16 mm to (225.9, 107.4)
- moved REF** 5.15 mm to (200.5, 92.5)
- moved U1 3.62 mm to (213.2, 99.8)
- moved SW1 2.84 mm to (210.7, 115.0)
- moved J3 0.19 mm to (242.4, 97.3)
Connections:
- Q1 pad 2: Net-(J2-Pin_1) -> /LED-
- R1 pad 2: Net-(U1-GPIO_7) -> Net-(U1-GPIO_8)
- R2 pad 2: Net-(U1-GPIO_8) -> Net-(U1-GPIO_9)
- SW1 pad A: Net-(U1-GPIO_7) -> Net-(U1-GPIO_8)
- SW1 pad B: Net-(U1-GPIO_8) -> Net-(U1-GPIO_9)
- U1 pad 14: Net-(SW2-B) -> /+5V_MCU
- U1 pad 2: unconnected-(U1-GPIO_17-Pad2) -> Net-(SW1-S2)
- U1 pad 3: Net-(SW1-S2) -> Net-(U1-GPIO_9)
- U1 pad 5: Net-(U1-GPIO_7) -> unconnected-(U1-GPIO_7-Pad5)
- U1 pad 6: unconnected-(U1-GPIO_6-Pad6) -> Net-(J3-ECHO)
- U1 pad 7: Net-(J3-ECHO) -> unconnected-(U1-GPIO_5-Pad7)
Routing:
- net Net-(SW2-B): track 40.9 -> 0.00 mm
- net /+24V: track 34.6 -> 0.01 mm
- net /+5V: track 17.4 -> 50.1 mm
- net Net-(U1-GPIO_7): track 27.5 -> 0.00 mm
- net /+5V_MCU: track 0.00 -> 23.4 mm
- net Net-(U1-GPIO_9): track 0.00 -> 20.6 mm
- net Net-(J3-Vcc): track 81.7 -> 99.8 mm
- net /+5V_SW: track 0.00 -> 15.0 mm
- net Net-(J2-Pin_1): track 13.5 -> 0.00 mm
- net Net-(U1-GPIO_8): track 19.9 -> 27.5 mm
- net Net-(J3-ECHO): track 11.2 -> 18.9 mm
- net Net-(J3-TRIG): track 20.9 -> 25.6 mm
- net Net-(U1-GPIO_18): track 36.2 -> 40.5 mm
- net Net-(Q1-G): track 8.89 -> 12.7 mm
- net Net-(SW1-S2): track 28.3 -> 27.8 mm
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- added copper zone on F.Cu, net /+24V
- added copper zone on F.Cu, net /LED-
- added copper zone on B.Cu, net <NO NET>
- added copper zone on F.Cu, net <NO NET>
- added copper zone on F.Cu, net Net-(J3-Vcc)
Other:
- board size 140 x 42 mm -> 150 x 42 mm
- board text added: "ADAFRUIT QTPy ESP32-S3"
- board text added: "CASE INTERIOR WALL"
- board text added: "INPUT: 5.1-36V MIN 500mA"
- board text added: "LID SCREW SPACE"
- board text added: "OUTPUT 5A MAX"
- board text removed: "3A MAX OUTPUT"
- board text removed: "<-POLOLU D24V10F5 24V>5V 1A"
- board text removed: "INPUT: 5.1-36V MIN 500mA MAX 3.5A"

Commit message: pcb board review
Parts:
- P1: renamed from Pololu_5V_1; value ~ -> Pololu D24V10F5
- S1: renamed from J3; value Screw_Terminal_HCSR04 -> RCWL-1601
- SW1: value Rotary Encoder (Quadrature) PEC11 -> PEC11
Connections:
- net Net-(J3-Vcc) renamed /+3V3
- J1 pad 1: /+24V -> <NO NET>
- J1 pad 2: <NO NET> -> /+24V
- P1 pad 1: unconnected-(Pololu_5V_1-PG-Pad1) -> (no net)
- P1 pad 2: unconnected-(Pololu_5V_1-SHDN-Pad2) -> (no net)
- P1 pad 3: /+24V -> (no net)
- P1 pad 4: <NO NET> -> (no net)
- P1 pad 5: /+5V -> (no net)
Other:
- board text added: "Hole for Case Mount"

Commit message: board updates
Parts:
- removed ?: Hole10mm, user:Hole10mm
- removed the REF** at (200.5, 92.5)
- P1: value Pololu D24V10F5 -> POLOLU D24V10F5
- moved D1 272.0 mm to (-68.4, 3.29)
- moved J1 272.0 mm to (-103.9, 26.1)
- moved J2 272.0 mm to (-103.9, 36.3)
- moved M3 272.0 mm to (-77.1, 31.2)
- moved P1 272.0 mm to (-105.2, 8.37)
- moved Q1 272.0 mm to (-94.4, 28.7)
- moved R1 272.0 mm to (-34.1, 37.6)
- moved R2 272.0 mm to (-34.1, 32.5)
- moved R3 272.0 mm to (-34.1, 27.4)
- moved R4 272.0 mm to (-80.5, 16.0)
- moved R5 272.0 mm to (-84.3, 16.0)
- moved REF** 272.0 mm to (-25.0, 29.0)
- moved REF** 272.0 mm to (-137.0, 6.00)
- moved S1 272.0 mm to (-17.6, 17.3)
- moved SW1 272.0 mm to (-49.3, 35.0)
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Connections:
- J1 pad 1: <NO NET> -> /+24V
- J1 pad 2: /+24V -> <NO NET>
- P1 pad 1: (no net) -> unconnected-(P1-PG-Pad1)
- P1 pad 2: (no net) -> unconnected-(P1-SHDN-Pad2)
- P1 pad 3: (no net) -> /+24V
- P1 pad 4: (no net) -> <NO NET>
- P1 pad 5: (no net) -> /+5V
Routing:
- net <NO NET>: track 0.01 -> 0.00 mm, vias 33 -> 31
Other:
- outline, holes or cut-outs redrawn
- board text added: "ADAFRUIT QTPY ESP32-S3"
- board text added: "JLCJLCJLCJLCJLC"
- board text added: "Ultrasonic Lighting Controler Designed by George Kuegler v1.0"
- board text removed: "ADAFRUIT QTPy ESP32-S3"
