File: kicad/board-layout/cablight.kicad_sch (KiCad schematic)
At the start: 13 parts, among them J1 Screw_Term_1x2_2.54mm, J2 Screw_Term_1x2_2.54mm, J3 Screw_Terminal_HCSR04, Q1 IRLB8721PBF, SW1 Rotary Encoder (Quadrature) P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, SW2 SW_SPST

Commit message: update board layout
Parts:
- removed SW2: SW_SPST, user:CUI_SPDT_500mA_3mm, symbol Switch:SW_SPST
- added D1: 1N5817, Diode_THT:D_DO-41_SOD81_P2.54mm_Vertical_KathodeUp, symbol Device:D
- added SW3: switch_SPDT_SLW_121586, user:CUI_SPDT_500mA_3mm, symbol user:switch_SPDT_SLW_121586
- added TP1: GND, TestPoint:TestPoint_Plated_Hole_D2.0mm, symbol Connector:TestPoint
- added TP2: 5V, TestPoint:TestPoint_Plated_Hole_D2.0mm, symbol Connector:TestPoint
- SW1: footprint user:Bourns-PEC11R-4220F-S0024-0-0-0 -> user:Bourns-PEC11R
Connections:
- net +5V: now also SW3.1, TP2.1
- net +5V_MCU: now reaches U1.14 (5V)
- net +5V_MCU: now also D1.1 (K)
- net at R3.2, SW1.2 (S2): now also U1.2 (GPIO_17); no longer U1.3 (GPIO_9)
- net at R1.2, SW1.A: now also U1.4 (GPIO_8); no longer U1.5 (GPIO_7)
- net at R2.2, SW1.B: now also U1.3 (GPIO_9); no longer U1.4 (GPIO_8)
- net at U1.6 (GPIO_6): now also J3.3 (ECHO)
- net at U1.7 (GPIO_5): no longer J3.3 (ECHO)
- net at J1.2 (Pin_2): now also TP1.1
- net LED-: now reaches J2.1 (Pin_1), Q1.2 (D)
- net GND: now reaches J3.4 (GND)
- new net +5V_SW: D1.2 (A), SW3.2
Other:
- moved on the sheet: R1, R2, R3, SW1

Commit message: pcb board review
Parts:
- P1: renamed from Pololu_5V_1; value ~ -> Pololu D24V10F5
- S1: renamed from J3; value Screw_Terminal_HCSR04 -> RCWL-1601; symbol Connector:Screw_Terminal_01x04 -> user:RCWL-1601
- SW1: value Rotary Encoder (Quadrature) PEC11 -> PEC11
Connections:
- net +24V: now also J1.2 (Pin_2), P1. (VOUT_5V); no longer J1.1 (Pin_1), P1.3 (VIN_24V)
- net +5V: now also P1. (VOUT_5V); no longer P1.5 (VOUT_5V)
- net at TP1.1: now also J1.1 (Pin_1); no longer J1.2 (Pin_2)
- net +3V3: now reaches R1.1, R2.1, R3.1, S1.1 (Vin), U1.12 (3.3V)
Other:
- title: (none) -> UNDERCABINET ULTRASONIC SENSOR
- moved on the sheet: D1, J1, R1, R2, R3, SW1, SW3, TP1, TP2

Commit message: board updates
Parts:
- P1: symbol Power Supply Module:Pololu_0J8557_24V -> user:Pololu_0J8557_24V
Connections:
- net +24V: now also J1.1 (Pin_1), P1.3 (VIN_24V); no longer J1.2 (Pin_2), P1. (VOUT_5V)
- net +5V: now also P1.5 (VOUT_5V); no longer P1. (VOUT_5V)
- net at TP1.1: now also J1.2 (Pin_2); no longer J1.1 (Pin_1)
Other:
- moved on the sheet: J1, J2, Q1, R4, R5, TP1
